File: hdw/minimal/minimal.kicad_sch (KiCad schematic)
At the start: 14 parts, among them J1 USB_A, SW1 RESET, SW2 BOOTLOADER, U1 CH552G

Commit message: doc - update
Parts:
- SW1: footprint Button_Switch_SMD:SW_SPST_Omron_B3FS-100xP -> Button_Switch_SMD:SW_SPST_SKQG_WithStem
- U1: footprint H_soic:SOIC16 -> Package_SO:SOIC-16W_5.3x10.2mm_P1.27mm
Changed lines of the file:
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@@
     (property "Reference" "SW1" (id 0) (at 134.7724 77.1144 0))
     (property "Value" "RESET" (id 1) (at 134.7724 79.6544 0))
-    (property "Footprint" "Button_Switch_SMD:SW_SPST_Omron_B3FS-100xP" (id 2) (at 134.7724 80.0608 0)
+    (property "Footprint" "Button_Switch_SMD:SW_SPST_SKQG_WithStem" (id 2) (at 134.7724 80.0608 0)
       (effects (font (size 1.27 1.27)) hide)
     )
@@
     (property "Reference" "U1" (id 0) (at 148.4376 80.9244 0))
     (property "Value" "CH552G" (id 1) (at 148.4376 83.4644 0))
-    (property "Footprint" "H_soic:SOIC16" (id 2) (at 148.4376 111.8616 0)
+    (property "Footprint" "Package_SO:SOIC-16W_5.3x10.2mm_P1.27mm" (id 2) (at 148.4376 111.8616 0)
       (effects (font (size 1.27 1.27)) hide)
     )
@@
     )
     (path "/c36d6a39-2caa-4975-a585-d762d089cd6d"
-      (reference "SW1") (unit 1) (value "RESET") (footprint "Button_Switch_SMD:SW_SPST_Omron_B3FS-100xP")
+      (reference "SW1") (unit 1) (value "RESET") (footprint "Button_Switch_SMD:SW_SPST_SKQG_WithStem")
     )
     (path "/21675d65-bdfb-4e9e-84c7-cd48b7855d37"
@@
     )
     (path "/c46fbcc7-964c-4651-a61c-9a277ad0e128"
-      (reference "U1") (unit 1) (value "CH552G") (footprint "H_soic:SOIC16")
+      (reference "U1") (unit 1) (value "CH552G") (footprint "Package_SO:SOIC-16W_5.3x10.2mm_P1.27mm")
     )
   )
