File: src/button_led_rgb/schematic.kicad_sch (KiCad schematic)
At the start: 5 parts, among them SW1 Push, U1 CH552G

Commit message: Save changes at: 1735251710
Parts:
- removed D1: LED, symbol Device:LED
- added LED: ~, LED_SMD:LED_ROHM_SMLVN6, symbol LED:SMLVN6RGB
Connections:
- net at R1.2: now also LED.4 (GK), LED.5 (RK), LED.6 (BK)
- net at U1.10 (P3.3): now also LED.2 (RA)
- net at U1.11 (P3.4): now also LED.1 (BA)
- net at U1.9 (P1.1): now also LED.3 (GA)
- no-connect marks 14 -> 12
Other:
- moved on the sheet: R1
Changed lines of the file:
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@@
+	)
+	(junction
+		(at 180.34 104.14)
+		(diameter 0)
+		(color 0 0 0 0)
 	)
 	(junction
@@
 	)
 	(no_connect
-		(at 162.56 104.14)
-	)
-	(no_connect
 		(at 162.56 99.06)
 	)
 	(no_connect
-		(at 162.56 101.6)
+		(at 134.62 106.68)
 	)
 	(no_connect
@@
 	)
 	(no_connect
-		(at 162.56 106.68)
-	)
-	(no_connect
 		(at 162.56 96.52)
 	)
 	(wire
 		(pts
-			(xy 124.46 106.68) (xy 121.92 106.68)
+			(xy 180.34 104.14) (xy 180.34 109.22)
+		)
+		(stroke
+			(width 0)
+			(type default)
+		)
+	)
+	(wire
+		(pts
+			(xy 162.56 101.6) (xy 165.1 101.6)
+		)
+		(stroke
+			(width 0)
+			(type default)
+		)
+	)
+	(wire
+		(pts
+			(xy 165.1 109.22) (xy 167.64 109.22)
+		)
+		(stroke
+			(width 0)
+			(type default)
+		)
+	)
+	(wire
+		(pts
+			(xy 190.5 104.14) (xy 193.04 104.14)
 		)
 		(stroke
@@
 	(wire
 		(pts
-			(xy 121.92 116.84) (xy 121.92 119.38)
-		)
-		(stroke
-			(width 0)
-			(type default)
-		)
-	)
-	(wire
-		(pts
-			(xy 132.08 106.68) (xy 134.62 106.68)
-		)
-		(stroke
-			(width 0)
-			(type default)
-		)
-	)
-	(wire
-		(pts
-			(xy 121.92 106.68) (xy 121.92 109.22)
+			(xy 162.56 104.14) (xy 167.64 104.14)
+		)
+		(stroke
+			(width 0)
+			(type default)
+		)
+	)
+	(wire
+		(pts
+			(xy 177.8 104.14) (xy 180.34 104.14)
+		)
+		(stroke
+			(width 0)
+			(type default)
+		)
+	)
+	(wire
+		(pts
+			(xy 177.8 99.06) (xy 180.34 99.06)
+		)
+		(stroke
+			(width 0)
+			(type default)
+		)
+	)
+	(wire
+		(pts
+			(xy 180.34 109.22) (xy 177.8 109.22)
 		)
 		(stroke
@@
 	(wire
 		(pts
+			(xy 180.34 99.06) (xy 180.34 104.14)
+		)
+		(stroke
+			(width 0)
+			(type default)
+		)
+	)
+	(wire
+		(pts
+			(xy 162.56 106.68) (xy 165.1 106.68)
+		)
+		(stroke
+			(width 0)
+			(type default)
+		)
+	)
+	(wire
+		(pts
+			(xy 180.34 104.14) (xy 182.88 104.14)
+		)
+		(stroke
+			(width 0)
+			(type default)
+		)
+	)
+	(wire
+		(pts
+			(xy 165.1 99.06) (xy 167.64 99.06)
+		)
+		(stroke
+			(width 0)
+			(type default)
+		)
+	)
+	(wire
+		(pts
 			(xy 121.92 76.2) (xy 121.92 78.74)
+		)
+		(stroke
+			(width 0)
+			(type default)
+		)
+	)
+	(wire
+		(pts
+			(xy 165.1 101.6) (xy 165.1 99.06)
+		)
+		(stroke
+			(width 0)
+			(type default)
+		)
+	)
+	(wire
+		(pts
+			(xy 165.1 106.68) (xy 165.1 109.22)
 		)
 		(stroke
@@
 	(symbol
 		(lib_id "power:GND")
-		(at 121.92 119.38 0)
+		(at 193.04 104.14 90)
 		(unit 1)
 		(exclude_from_sim no)
@@
 		(fields_autoplaced yes)
 		(property "Reference" "#PWR02"
-			(at 121.92 125.73 0)
+			(at 199.39 104.14 0)
 			(effects
 				(font
@@
 		)
 		(property "Value" "GND"
-			(at 121.92 124.46 0)
+			(at 198.12 104.14 0)
 			(effects
 				(font
@@
 		)
 		(property "Footprint" ""
-			(at 121.92 119.38 0)
+			(at 193.04 104.14 0)
 			(effects
 				(font
@@
 		)
 		(property "Datasheet" ""
-			(at 121.92 119.38 0)
+			(at 193.04 104.14 0)
 			(effects
 				(font
@@
 		)
 		(property "Description" ""
-			(at 121.92 119.38 0)
+			(at 193.04 104.14 0)
 			(effects
 				(font
@@
 	)
 	(symbol
-		(lib_id "Device:LED")
-		(at 128.27 106.68 0)
+		(lib_id "LED:SMLVN6RGB")
+		(at 172.72 104.14 0)
 		(unit 1)
 		(exclude_from_sim no)
@@
 		(on_board yes)
 		(dnp no)
-		(fields_autoplaced yes)
-		(property "Reference" "D1"
-			(at 126.6825 100.33 0)
-			(effects
-				(font
-					(size 1.27 1.27)
-				)
-			)
-		)
-		(property "Value" "LED"
-			(at 126.6825 102.87 0)
-			(effects
-				(font
-					(size 1.27 1.27)
-				)
-			)
-		)
-		(property "Footprint" ""
-			(at 128.27 106.68 0)
-			(effects
-				(font
-					(size 1.27 1.27)
-				)
-				(hide yes)
-			)
-		)
-		(property "Datasheet" "~"
-			(at 128.27 106.68 0)
-			(effects
-				(font
-					(size 1.27 1.27)
-				)
-				(hide yes)
-			)
-		)
-		(property "Description" ""
-			(at 128.27 106.68 0)
-			(effects
-				(font
-					(size 1.27 1.27)
-				)
-				(hide yes)
-			)
+		(property "Reference" "LED"
+			(at 172.72 94.234 0)
+			(effects
+				(font
+					(size 1.27 1.27)
+				)
+			)
+		)
+		(property "Value" "~"
+			(at 172.72 92.71 0)
+			(effects
+				(font
+					(size 1.27 1.27)
+				)
+			)
+		)
+		(property "Footprint" "LED_SMD:LED_ROHM_SMLVN6"
+			(at 172.72 113.03 0)
+			(effects
+				(font
+					(size 1.27 1.27)
+				)
+				(hide yes)
+			)
+		)
+		(property "Datasheet" "https://www.rohm.com/datasheet/SMLVN6RGB1U"
+			(at 172.72 105.41 0)
+			(effects
+				(font
+					(size 1.27 1.27)
+				)
+				(hide yes)
+			)
+		)
+		(property "Description" "High Brightness Tri-Color LED, RGB, 3.5x2.8mm"
+			(at 172.72 104.14 0)
+			(effects
+				(font
+					(size 1.27 1.27)
+				)
+				(hide yes)
+			)
+		)
+		(pin "3"
+		)
+		(pin "2"
 		)
 		(pin "1"
 		)
-		(pin "2"
+		(pin "5"
+		)
+		(pin "4"
+		)
+		(pin "6"
 		)
 		(instances
-			(project "schematic"
+			(project ""
 				(path "/e63e39d7-6ac0-4ffd-8aa3-1841a4541b55"
-					(reference "D1")
+					(reference "LED")
 					(unit 1)
 				)
@@
 	(symbol
 		(lib_id "Device:R")
-		(at 121.92 113.03 0)
+		(at 186.69 104.14 270)
 		(mirror x)
 		(unit 1)
@@
 		(dnp no)
 		(property "Reference" "R1"
-			(at 119.38 111.76 0)
+			(at 187.96 101.854 90)
 			(effects
 				(font
@@
 		)
 		(property "Value" "1k"
-			(at 119.38 114.3 0)
+			(at 187.96 106.68 90)
 			(effects
 				(font
@@
 		)
 		(property "Footprint" ""
-			(at 120.142 113.03 90)
+			(at 186.69 105.918 90)
 			(effects
 				(font
@@
 		)
 		(property "Datasheet" "~"
-			(at 121.92 113.03 0)
+			(at 186.69 104.14 0)
 			(effects
 				(font
@@
 		)
 		(property "Description" ""
-			(at 121.92 113.03 0)
-			(effects
-				(font
+			(at 186.69 104.14 0)
+			(effects
+				(font
