File: hdw/CH552G/CH552.kicad_sch (KiCad schematic)
At the start: 19 parts, among them J1 USB_A, J2 Conn_01x07, J3 Conn_01x07, SW1 RST, SW2 BOOT, U1 CH552G

Commit message: feat - breakout CH552G v2.0
Parts:
- removed D1, D2: LED, Library:L1206, symbol Device:LED
- removed H1, H2: MountingHole, MountingHole:MountingHole_2.2mm_M2, symbol Mechanical:MountingHole
- removed J1: USB_A, Library:USB_Micro-B, symbol Connector:USB_A
- removed J2: Conn_01x07, Connector_PinHeader_2.54mm:PinHeader_1x07_P2.54mm_Vertical, symbol Connector_Generic:Conn_01x07
- removed JP1: SolderJumper_2_Open, Library:SolderJumper, symbol Jumper:SolderJumper_2_Open
- removed R1, R4: 1k, Library:R1206, symbol Device:R
- added J1: Conn_01x08, Connector_PinHeader_2.54mm:PinHeader_1x08_P2.54mm_Vertical, symbol Connector_Generic:Conn_01x08
- added P1: USB_C_Plug_USB2.0, Library:USB_C_MC_112D, symbol Connector:USB_C_Plug_USB2.0
- SW1: value RST -> RESET
- renumbered D3 to D1, R2 to R1, R3 to R2
Connections:
- net +5V: now also J1.2 (Pin_2); no longer J3.1 (Pin_1)
- net GND: now also J1.1 (Pin_1), P1.A1 (GND), P1.A12 (GND), P1.B1 (GND), P1.B12 (GND); no longer J3.2 (Pin_2)
- net P1.1: now also J3.6 (Pin_6); no longer J3.7 (Pin_7)
- net P1.4: now also J1.5 (Pin_5)
- net P1.5: now also J1.4 (Pin_4)
- net P1.6: now also J1.7 (Pin_7)
- net P1.7: now also J1.8 (Pin_8)
- net P3.0: now also J3.2 (Pin_2)
- net P3.1: now also J3.1 (Pin_1)
- net P3.2: now also J1.6 (Pin_6)
- net P3.3: now also J3.7 (Pin_7); no longer J3.6 (Pin_6)
- net P3.6: now also P1.A6 (D+)
- net P3.7: now also P1.A7 (D-)
- net V33: now also J1.3 (Pin_3)
- net VBUS: now also P1.A4 (VBUS), P1.A9 (VBUS), P1.B4 (VBUS), P1.B9 (VBUS)
- no-connect marks 1 -> 3
Other:
- moved on the sheet: C1, C2, D1, F1, J3, R1, R2

Commit message: wip
Parts:
- removed F1: Polyfuse, Library:F1206, symbol Device:Polyfuse
- removed P1: USB_C_Plug_USB2.0, Library:USB_C_MC_112D, symbol Connector:USB_C_Plug_USB2.0
- added H1, H2, H3, H4: MountingHole, MountingHole:MountingHole_3.2mm_M3, symbol Mechanical:MountingHole
- added P1: USB_C_Receptacle_USB2.0, Library:USB_C_MC_112D, symbol Connector:USB_C_Receptacle_USB2.0
- D1: footprint Library:D1206 -> Library:SMA_DO_214AC
Connections:
- net +5V: now also D1.1 (K)
- net GND: now also P1.A1 (GND), P1.A12 (GND), P1.B1 (GND), P1.B12 (GND), P1.S1 (SHIELD)
- net P3.6: now also P1.A6 (D+), P1.B6 (D+)
- net P3.7: now also P1.A7 (D-), P1.B7 (D-)
- net VBUS: now also P1.A4 (VBUS), P1.A9 (VBUS), P1.B4 (VBUS), P1.B9 (VBUS)
- no-connect marks 3 -> 4
Other:
- moved on the sheet: D1

Commit message: Save changes at: 1734300643
Parts:
- added D2, D3: LED, Library:L1206, symbol Device:LED
- added R3, R4: 1k, Library:R1206, symbol Device:R
Connections:
- net +5V: now also R3.2
- net GND: now also D2.1 (K), D3.1 (K)
- net P3.0: now also R4.2
- new net: D2.2 (A), R3.1
- new net: D3.2 (A), R4.1

Commit message: Save changes at: 1734347778
Parts:
- removed J3: Conn_01x07, Connector_PinHeader_2.54mm:PinHeader_1x07_P2.54mm_Vertical, symbol Connector_Generic:Conn_01x07
- added J2: Conn_01x08, Connector_PinHeader_2.54mm:PinHeader_1x08_P2.54mm_Vertical, symbol Connector_Generic:Conn_01x08
- renumbered D2 to L1, D3 to L2, R3 to R1, R4 to R2, R1 to R3, R2 to R4
Connections:
- net +5V: now also SW1.1; no longer SW1.2
- net GND: now also J2.1 (Pin_1)
- net P1.1: now also J2.7 (Pin_7)
- net P3.0: now also J2.2 (Pin_2)
- net P3.1: now also J2.3 (Pin_3)
- net P3.3: now also J2.8 (Pin_8)
- net P3.4: now also J2.6 (Pin_6)
- net P3.6: now also J2.5 (Pin_5)
- net P3.7: now also J2.4 (Pin_4)
- net RST: now also SW1.2; no longer SW1.1
Changed lines of the file:
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@@
 	(global_label "P3.0"
 		(shape input)
-		(at 95.25 95.25 180)
+		(at 95.25 92.71 180)
 		(fields_autoplaced yes)
 		(effects
@@
 		)
 		(property "Intersheetrefs" "${INTERSHEET_REFS}"
-			(at 88.5431 95.1706 0)
+			(at 88.5431 92.6306 0)
 			(effects
 				(font
@@
 	(global_label "P3.1"
 		(shape input)
-		(at 95.25 92.71 180)
+		(at 95.25 95.25 180)
 		(fields_autoplaced yes)
 		(effects
@@
 		)
 		(property "Intersheetrefs" "${INTERSHEET_REFS}"
-			(at 88.5431 92.6306 0)
+			(at 88.5431 95.1706 0)
 			(effects
 				(font
@@
 	)
 	(symbol
-		(lib_id "Connector_Generic:Conn_01x07")
-		(at 100.33 100.33 0)
-		(unit 1)
-		(exclude_from_sim no)
-		(in_bom yes)
-		(on_board yes)
-		(dnp no)
-		(fields_autoplaced yes)
-		(property "Reference" "J3"
-			(at 102.87 99.0599 0)
-			(effects
-				(font
-					(size 1.27 1.27)
-				)
-				(justify left)
-			)
-		)
-		(property "Value" "Conn_01x07"
-			(at 102.87 101.5999 0)
-			(effects
-				(font
-					(size 1.27 1.27)
-				)
-				(justify left)
-			)
-		)
-		(property "Footprint" "Connector_PinHeader_2.54mm:PinHeader_1x07_P2.54mm_Vertical"
-			(at 100.33 100.33 0)
-			(effects
-				(font
-					(size 1.27 1.27)
-				)
-				(hide yes)
-			)
-		)
-		(property "Datasheet" "~"
-			(at 100.33 100.33 0)
-			(effects
-				(font
-					(size 1.27 1.27)
-				)
-				(hide yes)
-			)
-		)
-		(property "Description" ""
-			(at 100.33 100.33 0)
-			(effects
-				(font
-					(size 1.27 1.27)
-				)
-				(hide yes)
-			)
-		)
-		(pin "1"
-		)
-		(pin "2"
-		)
-		(pin "3"
-		)
-		(pin "4"
-		)
-		(pin "5"
-		)
-		(pin "6"
-		)
-		(pin "7"
-		)
-		(instances
-			(project "CH552"
-				(path "/e63e39d7-6ac0-4ffd-8aa3-1841a4541b55"
-					(reference "J3")
-					(unit 1)
-				)
-			)
-		)
-	)
-	(symbol
 		(lib_id "Connector:USB_C_Receptacle_USB2.0")
 		(at 208.28 102.87 0)
@@
 		(on_board yes)
 		(dnp no)
-		(property "Reference" "R2"
+		(property "Reference" "R4"
 			(at 161.29 53.7464 90)
 			(effects
@@
 			(project "CH552"
 				(path "/e63e39d7-6ac0-4ffd-8aa3-1841a4541b55"
-					(reference "R2")
+					(reference "R4")
 					(unit 1)
 				)
@@
 		(lib_id "Switch:SW_Push")
 		(at 149.86 45.72 0)
-		(unit 1)
-		(exclude_from_sim no)
-		(in_bom yes)
-		(on_board yes)
-		(dnp no)
-		(fields_autoplaced yes)
+		(mirror y)
+		(unit 1)
+		(exclude_from_sim no)
+		(in_bom yes)
+		(on_board yes)
+		(dnp no)
 		(property "Reference" "SW1"
 			(at 149.86 38.1 0)
@@
 				(path "/e63e39d7-6ac0-4ffd-8aa3-1841a4541b55"
 					(reference "#PWR0104")
+					(unit 1)
+				)
+			)
+		)
+	)
+	(symbol
+		(lib_id "Connector_Generic:Conn_01x08")
+		(at 100.33 97.79 0)
+		(unit 1)
+		(exclude_from_sim no)
+		(in_bom yes)
+		(on_board yes)
+		(dnp no)
+		(fields_autoplaced yes)
+		(property "Reference" "J2"
+			(at 102.87 97.79 0)
+			(effects
+				(font
+					(size 1.27 1.27)
+				)
+				(justify left)
+			)
+		)
+		(property "Value" "Conn_01x08"
+			(at 102.87 100.33 0)
+			(effects
+				(font
+					(size 1.27 1.27)
+				)
+				(justify left)
+			)
+		)
+		(property "Footprint" "Connector_PinHeader_2.54mm:PinHeader_1x08_P2.54mm_Vertical"
+			(at 100.33 97.79 0)
+			(effects
+				(font
+					(size 1.27 1.27)
+				)
+				(hide yes)
+			)
+		)
+		(property "Datasheet" "~"
+			(at 100.33 97.79 0)
+			(effects
+				(font
+					(size 1.27 1.27)
+				)
+				(hide yes)
+			)
+		)
+		(property "Description" ""
+			(at 100.33 97.79 0)
+			(effects
+				(font
+					(size 1.27 1.27)
+				)
+				(hide yes)
+			)
+		)
+		(pin "1"
+		)
+		(pin "2"
+		)
+		(pin "3"
+		)
+		(pin "4"
+		)
+		(pin "5"
+		)
+		(pin "6"
+		)
+		(pin "7"
+		)
+		(pin "8"
+		)
+		(instances
+			(project "CH552"
+				(path "/e63e39d7-6ac0-4ffd-8aa3-1841a4541b55"
+					(reference "J2")
 					(unit 1)
 				)
@@
 		(on_board yes)
 		(dnp no)
-		(property "Reference" "R3"
+		(property "Reference" "R1"
 			(at 153.67 123.5964 90)
 			(effects
@@
 			(project "CH552"
 				(path "/e63e39d7-6ac0-4ffd-8aa3-1841a4541b55"
-					(reference "R3")
+					(reference "R1")
 					(unit 1)
 				)
@@
 		(on_board yes)
 		(dnp no)
-		(property "Reference" "R4"
+		(property "Reference" "R2"
 			(at 153.67 136.2964 90)
 			(effects
@@
 			(project "CH552"
 				(path "/e63e39d7-6ac0-4ffd-8aa3-1841a4541b55"
-					(reference "R4")
+					(reference "R2")
 					(unit 1)
 				)
@@
 	)
 	(symbol
+		(lib_id "power:GND")
+		(at 95.25 90.17 270)
+		(unit 1)
+		(exclude_from_sim no)
+		(in_bom yes)
+		(on_board yes)
+		(dnp no)
+		(fields_autoplaced yes)
+		(property "Reference" "#PWR05"
+			(at 88.9 90.17 0)
+			(effects
+				(font
+					(size 1.27 1.27)
+				)
+				(hide yes)
+			)
+		)
+		(property "Value" "GND"
+			(at 91.0844 90.1699 90)
+			(effects
+				(font
+					(size 1.27 1.27)
+				)
+				(justify right)
+			)
+		)
+		(property "Footprint" ""
+			(at 95.25 90.17 0)
+			(effects
+				(font
+					(size 1.27 1.27)
+				)
+				(hide yes)
+			)
+		)
+		(property "Datasheet" ""
+			(at 95.25 90.17 0)
+			(effects
+				(font
+					(size 1.27 1.27)
+				)
+				(hide yes)
+			)
+		)
+		(property "Description" ""
+			(at 95.25 90.17 0)
+			(effects
+				(font
+					(size 1.27 1.27)
+				)
+				(hide yes)
+			)
+		)
+		(pin "1"
+		)
+		(instances
+			(project "CH552"
+				(path "/e63e39d7-6ac0-4ffd-8aa3-1841a4541b55"
+					(reference "#PWR05")
+					(unit 1)
+				)
+			)
+		)
+	)
+	(symbol
 		(lib_id "Device:LED")
 		(at 144.78 138.43 0)
@@
 		(dnp no)
 		(fields_autoplaced yes)
-		(property "Reference" "D3"
+		(property "Reference" "L2"
 			(at 143.1925 132.08 0)
 			(effects
@@
 			(project "CH552"
 				(path "/e63e39d7-6ac0-4ffd-8aa3-1841a4541b55"
-					(reference "D3")
+					(reference "L2")
 					(unit 1)
 				)
@@
 		(on_board yes)
 		(dnp no)
-		(property "Reference" "R1"
+		(property "Reference" "R3"
 			(at 149.86 67.31 90)
 			(effects
@@
 			(project "CH552"
 				(path "/e63e39d7-6ac0-4ffd-8aa3-1841a4541b55"
-					(reference "R1")
+					(reference "R3")
 					(unit 1)
 				)
@@
 		(dnp no)
 		(fields_autoplaced yes)
-		(property "Reference" "D2"
+		(property "Reference" "L1"
 			(at 143.1925 119.38 0)
 			(effects
@@
 			(project ""
 				(path "/e63e39d7-6ac0-4ffd-8aa3-1841a4541b55"
-					(reference "D2")
-					(unit 1)
-				)
+					(reference "L1")
+					(unit 1)
+				)

Commit message: Save changes at: 1734985773
Parts:
- added C3: 4700nF, Library:C1206, symbol Device:C
- added C4: 100nF, Library:C1206, symbol Device:C
- added F1: Polyfuse, Library:F1206, symbol Device:Polyfuse
- added R5, R6: 5.1k, Library:R1206, symbol Device:R
- P1: footprint Library:USB_C_MC_112D -> Connector_USB:USB_C_Receptacle_GCT_USB4105-xx-A_16P_TopMnt_Horizontal
Connections:
- net +5V: now also J2.2 (Pin_2), C3.1; no longer J1.2 (Pin_2)
- net GND: now also C3.2, C4.1, R5.2, R6.2
- net P1.1: now also J2.8 (Pin_8); no longer J2.7 (Pin_7)
- net P1.4: now also J1.3 (Pin_3); no longer J1.5 (Pin_5)
- net P1.6: now also J1.5 (Pin_5); no longer J1.7 (Pin_7)
- net P1.7: now also J1.6 (Pin_6); no longer J1.8 (Pin_8)
- net P3.0: now also J1.8 (Pin_8); no longer J2.2 (Pin_2)
- net P3.1: now also J1.7 (Pin_7); no longer J2.3 (Pin_3)
- net P3.2: now also J1.2 (Pin_2); no longer J1.6 (Pin_6)
- net P3.3: now also J2.7 (Pin_7); no longer J2.8 (Pin_8)
- net V33: now also J2.3 (Pin_3), C4.2; no longer J1.3 (Pin_3)
- net at P1.A5 (CC1): now also R5.1
- net at P1.B5 (CC2): now also R6.1
- net VBUS: no longer names the net of P1.A4 (VBUS), P1.A9 (VBUS), P1.B4 (VBUS), P1.B9 (VBUS)
- net VBUS: now also F1.1; no longer D1.2 (A)
- new net: D1.2 (A), F1.2
- no-connect marks 4 -> 2
Other:
- moved on the sheet: C1, C2, D1, J1, J2, L1, L2, P1, R1, R2, R3, R4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

Commit message: Save changes at: 1735508646
Parts:
- removed C4: 100nF, Library:C1206, symbol Device:C
Changed lines of the file:
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@@
-	)
-	(junction
-		(at 118.11 62.23)
-		(diameter 0)
-		(color 0 0 0 0)
 	)
 	(junction
@@
 	)
 	(junction
-		(at 127 85.09)
-		(diameter 0)
-		(color 0 0 0 0)
-	)
-	(junction
 		(at 95.25 102.87)
 		(diameter 0)
@@
 	(wire
 		(pts
-			(xy 127 85.09) (xy 129.54 85.09)
-		)
-		(stroke
-			(width 0)
-			(type default)
-		)
-	)
-	(wire
-		(pts
 			(xy 91.44 85.09) (xy 100.33 85.09)
 		)
@@
 	(wire
 		(pts
-			(xy 127 69.85) (xy 127 62.23)
-		)
-		(stroke
-			(width 0)
-			(type default)
-		)
-	)
-	(wire
-		(pts
 			(xy 95.25 102.87) (xy 124.46 102.87)
 		)
@@
 	(wire
 		(pts
-			(xy 127 77.47) (xy 127 85.09)
-		)
-		(stroke
-			(width 0)
-			(type default)
-		)
-	)
-	(wire
-		(pts
 			(xy 95.25 100.33) (xy 124.46 100.33)
 		)
@@
 	(wire
 		(pts
-			(xy 118.11 85.09) (xy 127 85.09)
+			(xy 118.11 85.09) (xy 129.54 85.09)
 		)
 		(stroke
@@
 		(pts
 			(xy 100.33 125.73) (xy 102.87 125.73)
-		)
-		(stroke
-			(width 0)
-			(type default)
-		)
-	)
-	(wire
-		(pts
-			(xy 127 62.23) (xy 118.11 62.23)
 		)
 		(stroke
@@
 					(unit 1)
 				)
-			)
-		)
-	)
-	(symbol
-		(lib_id "Device:C")
-		(at 127 73.66 0)
-		(mirror y)
-		(unit 1)
-		(exclude_from_sim no)
-		(in_bom yes)
-		(on_board yes)
-		(dnp no)
-		(property "Reference" "C4"
-			(at 125.73 74.93 90)
-			(effects
-				(font
-					(size 1.27 1.27)
-				)
-				(justify right)
-			)
-		)
-		(property "Value" "100nF"
-			(at 130.81 71.12 90)
-			(effects
-				(font
-					(size 1.27 1.27)
-				)
-				(justify right)
-			)
-		)
-		(property "Footprint" "Library:C1206"
-			(at 126.0348 77.47 0)
-			(effects
-				(font
-					(size 1.27 1.27)
-				)
-				(hide yes)
-			)
-		)
-		(property "Datasheet" "~"
-			(at 127 73.66 0)
-			(effects
-				(font
-					(size 1.27 1.27)
-				)
-				(hide yes)
-			)
-		)
-		(property "Description" ""
-			(at 127 73.66 0)
-			(effects
-				(font
-					(size 1.27 1.27)
-				)
-				(hide yes)
-			)
-		)
-		(pin "1"
-		)
-		(pin "2"
-		)
-		(instances
-			(project "CH552"
-				(path "/e63e39d7-6ac0-4ffd-8aa3-1841a4541b55"
-					(reference "C4")
-					(unit 1)
-				)
