File: hdw/CH552G/CH552.kicad_pcb (KiCad board)
At the start: 2 copper layers, 34.3 x 19.3 mm, 19 parts, among them J1 USB_A, J2 Conn_01x07, J3 Conn_01x07, SW1 RST, SW2 BOOT, U1 CH552G

Commit message: feat - breakout CH552G v2.0
Parts:
- removed the D1 at (158.8, 109.2)
- removed D2: LED, Library:L1206
- removed H1, H2: MountingHole, MountingHole:MountingHole_2.2mm_M2
- removed J2: Conn_01x07, Connector_PinHeader_2.54mm:PinHeader_1x07_P2.54mm_Vertical
- removed JP1: SolderJumper_2_Open, Library:SolderJumper
- removed the R1 at (158.8, 111.8)
- removed R4: 1k, Library:R1206
- added P1: USB_C_Plug_USB2.0, Library:USB_C_MC_112D, F.Cu at (132.7, 116.8)
- J1: value USB_A -> Conn_01x08; footprint Library:USB_Micro-B -> Connector_PinHeader_2.54mm:PinHeader_1x08_P2.54mm_Vertical
- SW1: value RST -> RESET
- moved C1 17.4 mm to (141.6, 120.0), turned to -90 degrees
- moved J3 15.4 mm to (154.3, 109.2)
- moved J1 8.03 mm to (136.5, 124.5), turned to 90 degrees
- moved R2 5.75 mm to (153.0, 120.0)
- moved R1 5.75 mm to (153.0, 113.7)
- moved C2 3.70 mm to (146.7, 120.0)
- moved F1 3.70 mm to (146.7, 116.8)
- moved D1 1.91 mm to (146.7, 113.7)
- moved U1 1.91 mm to (146.7, 116.8), turned to 180 degrees
- moved SW2 0.57 mm to (159.3, 119.8), turned to 180 degrees
- moved SW1 0.57 mm to (159.3, 113.9)
- renumbered D3 to D1, R2 to R1, R3 to R2
Connections:
- J1 pad 1: VBUS -> GND
- J1 pad 2: P3.7 -> +5V
- J1 pad 3: P3.6 -> V33
- J1 pad 4: GND -> P1.5
- J1 pad 5: unconnected-(J1-Shield-Pad5) -> P1.4
- J1 pad 6: (no net) -> P3.2
- J3 pad 1: +5V -> P3.1
- J3 pad 2: GND -> P3.0
- J3 pad 6: P3.3 -> P1.1
- J3 pad 7: P1.1 -> P3.3
Routing:
- net V33: track 15.8 -> 32.2 mm
- net VBUS: track 6.99 -> 18.7 mm
- net P1.4: track 18.4 -> 6.62 mm
- net Net-(D1-K): track 11.7 -> 3.17 mm
- net P1.7: track 6.31 -> 13.1 mm
- net Net-(D1-K) (its old number): track 6.49 -> 0.00 mm, vias 1 -> 0
- net Net-(D2-K): track 6.49 -> 0.00 mm, vias 1 -> 0
- net RST: track 27.2 -> 21.0 mm
- net P3.6: track 30.2 -> 36.1 mm
- net +5V: track 7.47 -> 13.2 mm, vias 1 -> 0
- net Net-(D1-A): track 5.22 -> 0.00 mm, vias 1 -> 0
- net P3.2: track 7.58 -> 3.20 mm
- net P1.5: track 5.41 -> 9.39 mm
- net P1.6: track 5.41 -> 9.29 mm
- net P3.7: track 18.2 -> 21.6 mm
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Other:
- board text added: "3.3V"
- board text added: "V2 2024/01"
- board text removed: "V1.1 2023/04"

Commit message: wip
Parts:
- removed F1: Polyfuse, Library:F1206
- added H1: MountingHole, MountingHole:MountingHole_3.2mm_M3, F.Cu at (132.1, 106.7)
- added H2: MountingHole, MountingHole:MountingHole_3.2mm_M3, F.Cu at (165.1, 106.7)
- added H3: MountingHole, MountingHole:MountingHole_3.2mm_M3, F.Cu at (165.1, 127.0)
- added H4: MountingHole, MountingHole:MountingHole_3.2mm_M3, F.Cu at (132.1, 127.0)
- C1, C2, R1, R2: moved to F.Cu
- D1: footprint Library:D1206 -> Library:SMA_DO_214AC; moved to F.Cu
- P1: value USB_C_Plug_USB2.0 -> USB_C_Receptacle_USB2.0
- moved D1 7.73 mm to (139.1, 112.4), turned to 90 degrees
- moved C2 7.00 mm to (139.7, 120.4), turned to 90 degrees
- moved J1 6.00 mm to (139.7, 129.5)
- moved J3 5.43 mm to (156.2, 104.1)
- moved SW2 4.66 mm to (163.8, 120.7)
- moved SW1 4.66 mm to (163.8, 113.0)
- moved R1 2.62 mm to (155.6, 113.0), turned to -90 degrees
- moved R2 2.62 mm to (155.6, 120.7), turned to -90 degrees
- moved U1 1.91 mm to (148.6, 116.8)
- moved C1 0.85 mm to (142.4, 120.4)
Connections:
- D1 pad 1: Net-(D1-K) -> +5V
- P1 pad A8: (no net) -> unconnected-(P1-SBU1-PadA8)
- P1 pad B6: (no net) -> P3.6
- P1 pad B7: (no net) -> P3.7
- P1 pad B8: (no net) -> unconnected-(P1-SBU2-PadB8)
- P1 pad S1: unconnected-(P1-SHIELD-PadS1) -> GND
Routing:
- net +5V: track 13.2 -> 0.00 mm
- net P3.6: track 36.1 -> 48.4 mm, vias 0 -> 1
- net V33: track 32.2 -> 41.7 mm
- net P3.7: track 21.6 -> 28.3 mm
- net VBUS: track 18.7 -> 12.0 mm
- net P3.2: track 3.20 -> 8.81 mm
- net P1.6: track 9.29 -> 14.6 mm
- net P3.4: track 8.05 -> 13.2 mm
- net P1.4: track 6.62 -> 11.3 mm
- net P1.7: track 13.1 -> 17.2 mm
- net P1.5: track 9.39 -> 13.3 mm
- net P3.3: track 9.29 -> 13.2 mm
- net P1.1: track 5.48 -> 9.33 mm
- net P3.0: track 5.48 -> 9.33 mm
- net P3.1: track 9.29 -> 12.7 mm
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Other:
- board size 34.3 x 19.3 mm -> 40.6 x 27.9 mm
- board text added: "V3.1 2024-04"
- board text added: "nicola@strappazzon.me"
- board text removed: "V2 2024/01"
- board text removed: "nstrappazzonc"

Commit message: Save changes at: 1734300643
Parts:
- added D2: LED, Library:L1206, F.Cu at (141.1, 108.2)
- added D3: LED, Library:L1206, F.Cu at (155.5, 108.2)
- added R3: 1k, Library:R1206, F.Cu at (141.1, 110.9)
- added R4: 1k, Library:R1206, F.Cu at (155.6, 110.9)
- moved D1 3.06 mm to (141.1, 114.7), turned to 0 degrees
- moved R2 2.67 mm to (156.7, 118.2), turned to 180 degrees
- moved R1 2.67 mm to (156.7, 115.4), turned to 0 degrees
- moved SW2 0.51 mm to (163.8, 120.1)
- moved SW1 0.51 mm to (163.8, 113.5)
- moved C1 0.05 mm to (142.4, 120.4)
- moved C2 0.05 mm to (139.8, 120.4)
Routing:
- net GND: track 12.4 -> 20.6 mm, vias 1 -> 2
- net P3.0: track 9.33 -> 13.5 mm
- net Net-(R2-Pad1): track 11.4 -> 8.58 mm
- net Net-(D2-A): track 0.00 -> 2.56 mm
- net P3.6: track 48.4 -> 46.9 mm
- net P3.1: track 12.7 -> 13.6 mm
- net P3.3: track 13.2 -> 13.8 mm

Commit message: Save changes at: 1734347778
Parts:
- removed J3: Conn_01x07, Connector_PinHeader_2.54mm:PinHeader_1x07_P2.54mm_Vertical
- added J2: Conn_01x08, Connector_PinHeader_2.54mm:PinHeader_1x08_P2.54mm_Vertical, F.Cu at (157.5, 104.1)
- moved R3 2.01 mm to (156.1, 113.5)
- moved R4 2.00 mm to (156.1, 120.1), turned to -90 degrees
- moved L2 0.53 mm to (156.1, 108.2)
- moved R2 0.53 mm to (156.1, 110.9)
- renumbered D2 to L1, D3 to L2, R3 to R1, R4 to R2, R1 to R3, R2 to R4
Connections:
- SW1 pad 1: RST -> +5V
- SW1 pad 2: +5V -> RST
Routing:
- net GND: track 20.6 -> 25.0 mm, vias 2 -> 1
- net Net-(L2-A): track 0.00 -> 2.70 mm
- net Net-(R4-Pad1): track 8.58 -> 11.0 mm
- net RST: track 17.6 -> 19.6 mm
- net P3.6: track 46.9 -> 48.8 mm
- net P3.1: track 13.6 -> 12.3 mm
- net P3.0: track 13.5 -> 14.5 mm
- net P3.7: track 28.3 -> 27.6 mm
- net P1.1: track 9.33 -> 9.86 mm
Other:
- board text added: "V3.2 2024-12"
- board text removed: "V3.1 2024-04"

Commit message: Save changes at: 1734985773
Parts:
- added C3: 4700nF, Library:C1206, F.Cu at (156.7, 109.4)
- added C4: 100nF, Library:C1206, F.Cu at (151.3, 109.5)
- added F1: Polyfuse, Library:F1206, F.Cu at (140.3, 124.2)
- added R5: 5.1k, Library:R1206, F.Cu at (140.3, 112.0)
- added R6: 5.1k, Library:R1206, F.Cu at (140.3, 121.7)
- P1: footprint Library:USB_C_MC_112D -> Connector_USB:USB_C_Receptacle_GCT_USB4105-xx-A_16P_TopMnt_Horizontal
- moved J2 17.8 mm to (139.7, 104.1), turned to 90 degrees
- moved L2 16.2 mm to (158.6, 124.2), turned to 180 degrees
- moved R2 13.7 mm to (153.2, 124.2)
- moved C2 12.5 mm to (145.8, 109.4), turned to 180 degrees
- moved C1 11.2 mm to (140.3, 109.4), turned to 180 degrees
- moved D1 11.1 mm to (146.8, 124.2)
- moved L1 8.87 mm to (139.1, 116.8), turned to -90 degrees
- moved SW1 6.37 mm to (164.3, 119.9)
- moved SW2 6.37 mm to (164.3, 113.8)
- moved R4 6.35 mm to (156.0, 113.8)
- moved R3 6.35 mm to (156.0, 119.9), turned to 90 degrees
- moved R1 6.00 mm to (141.7, 116.8), turned to 90 degrees
- moved P1 0.76 mm to (132.0, 116.8)
- turned U1 to 90 degrees
Connections:
- D1 pad 2: VBUS -> Net-(D1-A)
- J1 pad 2: +5V -> P3.2
- J1 pad 3: V33 -> P1.4
- J1 pad 5: P1.4 -> P1.6
- J1 pad 6: P3.2 -> P1.7
- J1 pad 7: P1.6 -> P3.1
- J1 pad 8: P1.7 -> P3.0
- J2 pad 2: P3.0 -> +5V
- J2 pad 3: P3.1 -> V33
- J2 pad 7: P1.1 -> P3.3
- J2 pad 8: P3.3 -> P1.1
- P1 pad A4: VBUS -> Net-(F1-Pad1)
- P1 pad A5: unconnected-(P1-CC1-PadA5) -> Net-(P1-CC1)
- P1 pad A9: VBUS -> Net-(F1-Pad1)
- P1 pad B4: VBUS -> Net-(F1-Pad1)
- P1 pad B5: unconnected-(P1-CC2-PadB5) -> Net-(P1-CC2)
- P1 pad B9: VBUS -> Net-(F1-Pad1)
Routing:
- net V33: track 42.1 -> 60.3 mm, vias 1 -> 3
- net Net-(P1-CC1): track 0.00 -> 15.1 mm, vias 0 -> 2
- net Net-(P1-CC2): track 0.00 -> 14.6 mm, vias 0 -> 2
- net Net-(F1-Pad1): track 0.00 -> 14.1 mm
- net VBUS: track 11.9 -> 0.00 mm
- net P3.7: track 27.6 -> 33.5 mm, vias 0 -> 2
- net P1.1: track 9.86 -> 15.5 mm, vias 0 -> 1
- net P3.2: track 8.81 -> 14.4 mm, vias 0 -> 1
- net Net-(D1-A): track 0.00 -> 2.78 mm
- net P3.0: track 14.5 -> 17.2 mm, vias 0 -> 2
- net P3.1: track 12.3 -> 15.0 mm, vias 0 -> 1
- net P1.4: track 11.3 -> 13.9 mm, vias 0 -> 1
- net P1.7: track 17.2 -> 15.0 mm, vias 0 -> 1
- net P3.6: track 48.8 -> 47.5 mm, vias 1 -> 3
- net P3.4: track 13.5 -> 14.4 mm, vias 0 -> 1
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
Commit message: Save changes at: 1735434824
Other:
- board text added: "3V3"
- board text removed: "3.3V"
Changed lines of the file:
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@@
 		)
 		(property "Footprint" "Library:R1206"
-			(at 0 0 360)
+			(at 0 0 0)
 			(layer "F.Fab")
 			(hide yes)
@@
 		)
 		(property "Datasheet" ""
-			(at 0 0 360)
+			(at 0 0 0)
 			(layer "F.Fab")
 			(hide yes)
@@
 		)
 		(property "Description" ""
-			(at 0 0 360)
+			(at 0 0 0)
 			(layer "F.Fab")
 			(hide yes)
@@
 		)
 		(property "Footprint" "Library:L1206"
-			(at 0 0 360)
+			(at 0 0 0)
 			(layer "F.Fab")
 			(hide yes)
@@
 		)
 		(property "Datasheet" ""
-			(at 0 0 360)
+			(at 0 0 0)
 			(layer "F.Fab")
 			(hide yes)
@@
 		)
 		(property "Description" "Light emitting diode"
-			(at 0 0 360)
+			(at 0 0 0)
 			(layer "F.Fab")
 			(hide yes)
@@
 		)
 		(fp_text user "${REFERENCE}"
-			(at 0 -3.6 360)
+			(at 0 -3.6 0)
 			(layer "F.Fab")
 			(hide yes)
@@
 		)
 	)
-	(gr_text "3.3V"
+	(gr_text "3V3"
 		(at 144.78 106.172 180)
 		(layer "F.SilkS")

Commit message: Save changes at: 1735508646
Parts:
- removed C4: 100nF, Library:C1206
- moved C3 5.46 mm to (151.3, 109.4), turned to 0 degrees
Routing:
- net GND: track 24.7 -> 30.1 mm, vias 6 -> 5
- net V33: track 60.3 -> 56.6 mm

Commit message: Save changes at: 1738020124
Parts:
- SW1: value RESET -> RST
- SW2: value BOOT -> BL
- moved SW1 0.90 mm to (163.4, 120.0)
- moved SW2 0.90 mm to (163.4, 113.7)
- moved D1 0.25 mm to (146.8, 124.5)
- moved F1 0.25 mm to (140.3, 124.5)
- moved L2 0.25 mm to (158.6, 124.5)
- moved R2 0.25 mm to (153.2, 124.5)
- moved C1 0.21 mm to (140.3, 109.2)
- moved C2 0.21 mm to (145.8, 109.2)
- moved C3 0.21 mm to (151.3, 109.2)
Routing:
- net GND: track 30.1 -> 35.0 mm, vias 5 -> 4
- net P3.0: track 17.2 -> 18.8 mm
- net V33: track 56.6 -> 57.7 mm
- net P3.6: track 47.5 -> 48.4 mm
- net Net-(R4-Pad1): track 11.7 -> 12.2 mm
- net P1.7: track 15.0 -> 15.5 mm
Other:
- board text added: "V3.3 2025-01"
- board text removed: "V3.2 2024-12"
