File: hdw/USBC2/USBC2.kicad_pcb (KiCad board)
At the start: 2 copper layers, 14 x 17.8 mm, 7 parts, among them J1 Conn_01x02, J2 Conn_01x02, J3 Conn_01x02, J4 Conn_01x02, P1 USB_C_Receptacle_USB2.0

Commit message: Save changes at: 1736461490
Other:
- board text added: "D+"
- board text added: "D-"
- board text removed: "D"
